File: elec/RollingBaseBoard/Com.sch (KiCad schematic (older format))
At the start: 9 parts, among them P10 UART_2, P11 I2C, P9 UART_1

Commit message: Updated the schematics to use the proper footprints.
Also regenerated the net list file.
Parts:
- P10, P11, P9: footprint (none) -> Footprints:Conn_01x03
- R18, R19, R20, R21, R22, R23: footprint (none) -> Footprints:R_CMS1206
Changed lines of the file:
@@
 F 0 "P9" H 6450 3700 50  0000 C CNN
 F 1 "UART_1" V 6550 3500 50  0000 C CNN
-F 2 "" H 6450 3500 60  0000 C CNN
+F 2 "Footprints:Conn_01x03" H 6450 3500 60  0001 C CNN
 F 3 "" H 6450 3500 60  0000 C CNN
 	1    6450 3500
@@
 F 0 "P10" H 6450 4250 50  0000 C CNN
 F 1 "UART_2" V 6550 4050 50  0000 C CNN
-F 2 "" H 6450 4050 60  0000 C CNN
+F 2 "Footprints:Conn_01x03" H 6450 4050 60  0001 C CNN
 F 3 "" H 6450 4050 60  0000 C CNN
 	1    6450 4050
@@
 F 0 "P11" H 6450 4800 50  0000 C CNN
 F 1 "I2C" V 6550 4600 50  0000 C CNN
-F 2 "" H 6450 4600 60  0000 C CNN
+F 2 "Footprints:Conn_01x03" H 6450 4600 60  0001 C CNN
 F 3 "" H 6450 4600 60  0000 C CNN
 	1    6450 4600
@@
 F 0 "R18" V 5280 2800 50  0000 C CNN
 F 1 "10kΩ" V 5200 2800 50  0000 C CNN
-F 2 "" V 5130 2800 30  0000 C CNN
+F 2 "Footprints:R_CMS1206" V 5130 2800 30  0001 C CNN
 F 3 "" H 5200 2800 30  0000 C CNN
 	1    5200 2800
@@
 F 0 "R19" V 5480 2800 50  0000 C CNN
 F 1 "10kΩ" V 5400 2800 50  0000 C CNN
-F 2 "" V 5330 2800 30  0000 C CNN
+F 2 "Footprints:R_CMS1206" V 5330 2800 30  0001 C CNN
 F 3 "" H 5400 2800 30  0000 C CNN
 	1    5400 2800
@@
 F 0 "R20" V 5680 2800 50  0000 C CNN
 F 1 "10kΩ" V 5600 2800 50  0000 C CNN
-F 2 "" V 5530 2800 30  0000 C CNN
+F 2 "Footprints:R_CMS1206" V 5530 2800 30  0001 C CNN
 F 3 "" H 5600 2800 30  0000 C CNN
 	1    5600 2800
@@
 F 0 "R21" V 5880 2800 50  0000 C CNN
 F 1 "10kΩ" V 5800 2800 50  0000 C CNN
-F 2 "" V 5730 2800 30  0000 C CNN
+F 2 "Footprints:R_CMS1206" V 5730 2800 30  0001 C CNN
 F 3 "" H 5800 2800 30  0000 C CNN
 	1    5800 2800
@@
 F 0 "R22" V 6080 2800 50  0000 C CNN
 F 1 "10kΩ" V 6000 2800 50  0000 C CNN
-F 2 "" V 5930 2800 30  0000 C CNN
+F 2 "Footprints:R_CMS1206" V 5930 2800 30  0001 C CNN
 F 3 "" H 6000 2800 30  0000 C CNN
 	1    6000 2800
@@
 F 0 "R23" V 6280 2800 50  0000 C CNN
 F 1 "10kΩ" V 6200 2800 50  0000 C CNN
-F 2 "" V 6130 2800 30  0000 C CNN
+F 2 "Footprints:R_CMS1206" V 6130 2800 30  0001 C CNN
 F 3 "" H 6200 2800 30  0000 C CNN
 	1    6200 2800
