File: elec/RollingBaseBoard/Driver.sch (KiCad schematic (older format))
At the start: 10 parts, among them P12 Motor, U1 LMD18201

Commit message: Updated the schematics to use the proper footprints.
Also regenerated the net list file.
Parts:
- C11, C13, C14, C15: footprint (none) -> Footprints:C_CMS0603
- C12: footprint (none) -> Footprints:C_CMS1210
- CP1: footprint (none) -> Footprints:C_Radial
- P12: footprint (none) -> Footprints:Power_Conn_01x02
- R24, R25: footprint (none) -> Footprints:R_CMS1206
- U1: footprint (none) -> Footprints:LMD18201
Changed lines of the file:
@@
 F 0 "U2" H 7100 3050 60  0000 C CNN
 F 1 "LMD18201" H 7100 4350 60  0000 C CNN
-F 2 "" H 6950 4500 60  0000 C CNN
+F 2 "Footprints:LMD18201" H 6950 4500 60  0001 C CNN
 F 3 "" H 6950 4500 60  0000 C CNN
 	1    7100 3700
@@
 F 0 "P13" H 5600 2750 50  0000 C CNN
 F 1 "Motor" V 5700 2600 50  0000 C CNN
-F 2 "" H 5600 2600 60  0000 C CNN
+F 2 "Footprints:Power_Conn_01x02" H 5600 2600 60  0001 C CNN
 F 3 "" H 5600 2600 60  0000 C CNN
 	1    5600 2600
@@
 F 0 "C19" H 6325 3250 50  0000 L CNN
 F 1 "10nF" H 6325 3050 50  0000 L CNN
-F 2 "" H 6338 3000 30  0000 C CNN
+F 2 "Footprints:C_CMS0603" H 6338 3000 30  0001 C CNN
 F 3 "" H 6300 3150 60  0000 C CNN
 	1    6300 3150
@@
 F 0 "C20" H 6325 4350 50  0000 L CNN
 F 1 "10nF" H 6325 4150 50  0000 L CNN
-F 2 "" H 6338 4100 30  0000 C CNN
+F 2 "Footprints:C_CMS0603" H 6338 4100 30  0001 C CNN
 F 3 "" H 6300 4250 60  0000 C CNN
 	1    6300 4250
@@
 F 0 "C16" H 4025 3850 50  0000 L CNN
 F 1 "100nF" H 4025 3650 50  0000 L CNN
-F 2 "" H 4038 3600 30  0000 C CNN
+F 2 "Footprints:C_CMS0603" H 4038 3600 30  0001 C CNN
 F 3 "" H 4000 3750 60  0000 C CNN
 	1    4000 3750
@@
 F 0 "C17" H 4325 3850 50  0000 L CNN
 F 1 "10µF" H 4325 3650 50  0000 L CNN
-F 2 "" H 4338 3600 30  0000 C CNN
+F 2 "Footprints:C_CMS1210" H 4338 3600 30  0001 C CNN
 F 3 "" H 4300 3750 60  0000 C CNN
 	1    4300 3750
@@
 F 0 "CP2" H 4675 3850 50  0000 L CNN
 F 1 "330µF" H 4675 3650 50  0000 L CNN
-F 2 "" H 4650 3750 60  0000 C CNN
+F 2 "Footprints:C_Radial" H 4650 3750 60  0001 C CNN
 F 3 "" H 4650 3750 60  0000 C CNN
 	1    4650 3750
@@
 F 0 "R26" V 5030 4050 50  0000 C CNN
 F 1 "10kΩ" V 4950 4050 50  0000 C CNN
-F 2 "" V 4880 4050 30  0000 C CNN
+F 2 "Footprints:R_CMS1206" V 4880 4050 30  0001 C CNN
 F 3 "" H 4950 4050 30  0000 C CNN
 	1    4950 4050
@@
 F 0 "R27" V 5230 4050 50  0000 C CNN
 F 1 "10kΩ" V 5150 4050 50  0000 C CNN
-F 2 "" V 5080 4050 30  0000 C CNN
+F 2 "Footprints:R_CMS1206" V 5080 4050 30  0001 C CNN
 F 3 "" H 5150 4050 30  0000 C CNN
 	1    5150 4050
@@
 F 0 "C18" H 5625 3200 50  0000 L CNN
 F 1 "1nF" H 5625 3000 50  0000 L CNN
-F 2 "" H 5638 2950 30  0000 C CNN
+F 2 "Footprints:C_CMS0603" H 5638 2950 30  0001 C CNN
 F 3 "" H 5600 3100 60  0000 C CNN
 	1    5600 3100
