File: elec/RollingBaseBoard/GP2.sch (KiCad schematic (older format))
At the start: 5 parts, among them P1 GP2

Commit message: Updated the schematics to use the proper footprints.
Also regenerated the net list file.
Parts:
- C1: footprint (none) -> Footprints:C_CMS1210
- C2: footprint (none) -> Footprints:C_CMS0603
- P1: footprint (none) -> Footprints:Conn_01x03
- R2, R3: footprint (none) -> Footprints:R_CMS1206
Changed lines of the file:
@@
 F 0 "P4" H 4900 3950 50  0000 C CNN
 F 1 "GP2" V 5000 3750 50  0000 C CNN
-F 2 "" H 4900 3750 60  0000 C CNN
+F 2 "Footprints:Conn_01x03" H 4900 3750 60  0001 C CNN
 F 3 "" H 4900 3750 60  0000 C CNN
 	1    4900 3750
@@
 F 0 "C7" H 5275 3550 50  0000 L CNN
 F 1 "10µF" H 5275 3350 50  0000 L CNN
-F 2 "" H 5288 3300 30  0000 C CNN
+F 2 "Footprints:C_CMS1210" H 5288 3300 30  0001 C CNN
 F 3 "" H 5250 3450 60  0000 C CNN
 	1    5250 3450
@@
 F 0 "R8" V 5780 3850 50  0000 C CNN
 F 1 "10kΩ" V 5700 3850 50  0000 C CNN
-F 2 "" V 5630 3850 30  0000 C CNN
+F 2 "Footprints:R_CMS1206" V 5630 3850 30  0001 C CNN
 F 3 "" H 5700 3850 30  0000 C CNN
 	1    5700 3850
@@
 F 0 "R9" V 6280 3850 50  0000 C CNN
 F 1 "20kΩ" V 6200 3850 50  0000 C CNN
-F 2 "" V 6130 3850 30  0000 C CNN
+F 2 "Footprints:R_CMS1206" V 6130 3850 30  0001 C CNN
 F 3 "" H 6200 3850 30  0000 C CNN
 	1    6200 3850
@@
 F 0 "C8" H 5975 3750 50  0000 L CNN
 F 1 "100nF" H 5975 3550 50  0000 L CNN
-F 2 "" H 5988 3500 30  0000 C CNN
+F 2 "Footprints:C_CMS0603" H 5988 3500 30  0001 C CNN
 F 3 "" H 5950 3650 60  0000 C CNN
 	1    5950 3650
