File: elec/RollingBaseBoard/Power.sch (KiCad schematic (older format))
At the start: 3 parts, among them P5 Bat5V, P6 Bat15V

Commit message: Updated the schematics to use the proper footprints.
Also regenerated the net list file.
Parts:
- F1: footprint (none) -> Footprints:Fuse
- P5: footprint (none) -> Footprints:Conn_01x02
- P6: footprint (none) -> Footprints:Power_Conn_01x02
Changed lines of the file:
@@
 F 0 "P5" H 5150 3350 50  0000 C CNN
 F 1 "Bat5V" V 5250 3200 50  0000 C CNN
-F 2 "" H 5150 3200 60  0000 C CNN
+F 2 "Footprints:Conn_01x02" H 5150 3200 60  0001 C CNN
 F 3 "" H 5150 3200 60  0000 C CNN
 	1    5150 3200
@@
 F 0 "P6" H 6800 3350 50  0000 C CNN
 F 1 "Bat15V" V 6900 3200 50  0000 C CNN
-F 2 "" H 6800 3200 60  0000 C CNN
+F 2 "Footprints:Power_Conn_01x02" H 6800 3200 60  0001 C CNN
 F 3 "" H 6800 3200 60  0000 C CNN
 	1    6800 3200
@@
 F 0 "F1" H 5800 3750 50  0000 C CNN
 F 1 "FUSE" H 5600 3650 50  0000 C CNN
-F 2 "" H 5700 3700 60  0000 C CNN
+F 2 "Footprints:Fuse" H 5700 3700 60  0001 C CNN
 F 3 "" H 5700 3700 60  0000 C CNN
 	1    5700 3700
