File: elec/RollingBaseBoard/RollingBaseBoard.sch (KiCad schematic (older format))
At the start: 1 part

Commit message: Updated the schematics to use the proper footprints.
Also regenerated the net list file.
Parts:
- R1: footprint (none) -> Footprints:R_CMS1206
Changed lines of the file:
@@
 F 0 "R1" V 5980 5850 50  0000 C CNN
 F 1 "10kΩ" V 5900 5850 50  0000 C CNN
-F 2 "" V 5830 5850 30  0000 C CNN
+F 2 "Footprints:R_CMS1206" V 5830 5850 30  0001 C CNN
 F 3 "" H 5900 5850 30  0000 C CNN
 	1    5900 5850
