File: elec/RollingBaseBoard/SwitchInput.sch (KiCad schematic (older format))
At the start: 4 parts, among them P16 Switch

Commit message: Updated the schematics to use the proper footprints.
Also regenerated the net list file.
Parts:
- C21: footprint (none) -> Footprints:C_CMS0603
- P16: footprint (none) -> Footprints:Conn_01x02
- R33, R34: footprint (none) -> Footprints:R_CMS1206
Changed lines of the file:
@@
 F 0 "R41" V 5780 3350 50  0000 C CNN
 F 1 "100kΩ" V 5700 3350 50  0000 C CNN
-F 2 "" V 5630 3350 30  0000 C CNN
+F 2 "Footprints:R_CMS1206" V 5630 3350 30  0001 C CNN
 F 3 "" H 5700 3350 30  0000 C CNN
 	1    5700 3350
@@
 F 0 "R42" V 6030 3500 50  0000 C CNN
 F 1 "18kΩ" V 5950 3500 50  0000 C CNN
-F 2 "" V 5880 3500 30  0000 C CNN
+F 2 "Footprints:R_CMS1206" V 5880 3500 30  0001 C CNN
 F 3 "" H 5950 3500 30  0000 C CNN
 	1    5950 3500
@@
 F 0 "C25" H 6175 3850 50  0000 L CNN
 F 1 "1µF" H 6175 3650 50  0000 L CNN
-F 2 "" H 6188 3600 30  0000 C CNN
+F 2 "Footprints:C_CMS0603" H 6188 3600 30  0001 C CNN
 F 3 "" H 6150 3750 60  0000 C CNN
 	1    6150 3750
@@
 F 0 "P20" H 5500 4000 50  0000 C CNN
 F 1 "Switch" V 5600 3850 50  0000 C CNN
-F 2 "" H 5500 3850 60  0000 C CNN
+F 2 "Footprints:Conn_01x02" H 5500 3850 60  0001 C CNN
 F 3 "" H 5500 3850 60  0000 C CNN
 	1    5500 3850
